Commit message: added/tested gripper urdf and collision sphere code

File: content/assets/urdf/robot_info/robot.urdf (robot description, URDF)
Before this commit: robot ur, 13 links, 12 joints
Links:
- added link left_bar, mass 0.022614240507152; collision mesh filename=robotiq_2f_85_gripper_visualization/meshes/collision/bar.stl; visual mesh filename=robotiq_2f_85_gripper_visualization/meshes/visual/bar.stl
- added link left_distal_phalanx, mass 0.0104003125914103; collision mesh filename=robotiq_2f_85_gripper_visualization/meshes/collision/distal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; visual mesh filename=robotiq_2f_85_gripper_visualization/meshes/visual/distal_ph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
- added link left_outer_knuckle, mass 0.00853198276973456; collision mesh filename=robotiq_2f_85_gripper_visualization/meshes/collision/outer_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; visual mesh filename=robotiq_2f_85_gripper_visualization/meshes/visual/outer_knu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
- added link left_proximal_phalanx, mass 0.0271177346495152; collision mesh filename=robotiq_2f_85_gripper_visualization/meshes/collision/proxim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; visual mesh filename=robotiq_2f_85_gripper_visualization/meshes/visual/proximal_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
- added link right_bar, mass 0.022614240507152; collision mesh filename=robotiq_2f_85_gripper_visualization/meshes/collision/bar.stl; visual mesh filename=robotiq_2f_85_gripper_visualization/meshes/visual/bar.stl
- added link right_distal_phalanx, mass 0.0104003125914103; collision mesh filename=robotiq_2f_85_gripper_visualization/meshes/collision/distal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; visual mesh filename=robotiq_2f_85_gripper_visualization/meshes/visual/distal_ph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
- added link right_outer_knuckle, mass 0.00853198276973456; collision mesh filename=robotiq_2f_85_gripper_visualization/meshes/collision/outer_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; visual mesh filename=robotiq_2f_85_gripper_visualization/meshes/visual/outer_knu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
- added link right_proximal_phalanx, mass 0.0271177346495152; collision mesh filename=robotiq_2f_85_gripper_visualization/meshes/collision/proxim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; visual mesh filename=robotiq_2f_85_gripper_visualization/meshes/visual/proximal_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
- added link robotiq_arg2f_base_link, mass 0.7; collision mesh filename=robotiq_2f_85_gripper_visualization/meshes/collision/base_l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; visual mesh filename=robotiq_2f_85_gripper_visualization/meshes/visual/base_link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
Joints:
- added joint gripper_main_joint: type fixed, parent wrist_3_link, child robotiq_arg2f_base_link, origin xyz=0 0 0 rpy=0 0 90
- added joint left_bar_joint: type fixed, parent left_distal_phalanx, child left_bar, origin xyz=0 0.0315 -0.0041 rpy=0 0 0, axis 1 0 0
- added joint left_distal_phalanx_joint: type fixed, parent left_proximal_phalanx, child left_distal_phalanx, origin xyz=0 0.0061 0.0471 rpy=0 0 0, axis 0 0 0, limit lower=-0.8757 upper=0 effort=1000 velocity=0.5, mimic joint=left_outer_knuckle_joint multiplier=-1 offset=0
- added joint left_outer_knuckle_joint: type fixed, parent robotiq_arg2f_base_link, child left_outer_knuckle, origin xyz=0 -0.0306011 0.054904 rpy=0 0 3.141592653589793, axis 0 0 0, limit lower=0 upper=0.8 effort=1000 velocity=0.5
- added joint left_proximal_phalanx_joint: type fixed, parent robotiq_arg2f_base_link, child left_proximal_phalanx, origin xyz=0 -0.0127 0.06142 rpy=.125 0 3.141592653589793, axis 1 0 0, limit lower=0 upper=0.8757 effort=1000 velocity=0.5, mimic joint=left_outer_knuckle_joint multiplier=1 offset=0
- added joint right_bar_joint: type fixed, parent right_distal_phalanx, child right_bar, origin xyz=0 0.0315 -0.0041 rpy=0 0 0, axis 1 0 0
- added joint right_distal_phalanx_joint: type fixed, parent right_proximal_phalanx, child right_distal_phalanx, origin xyz=0 0.0061 0.0471 rpy=0 0 0, axis 1 0 0, limit lower=-0.8757 upper=0 effort=1000 velocity=0.5, mimic joint=left_outer_knuckle_joint multiplier=-1 offset=0
- added joint right_outer_knuckle_joint: type fixed, parent robotiq_arg2f_base_link, child right_outer_knuckle, origin xyz=0 0.0306011 0.054904 rpy=0 0 0, axis 1 0 0, limit lower=0 upper=0.81 effort=1000 velocity=0.5, mimic joint=left_outer_knuckle_joint multiplier=1 offset=0
- added joint right_proximal_phalanx_joint: type fixed, parent robotiq_arg2f_base_link, child right_proximal_phalanx, origin xyz=0 0.0127 0.06142 rpy=.125 0 0.0, axis 1 0 0, limit lower=0 upper=0.8757 effort=1000 velocity=0.5, mimic joint=left_outer_knuckle_joint multiplier=1 offset=0

File: content/assets/urdf/robot_info/robot_storm.urdf (robot description, URDF)
Before this commit: robot ur, 7 links, 6 joints
Links:
- added link gripper_link, mass 0.7; collision mesh filename=robotiq_2f_85_gripper_visualization/meshes/collision/base_l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; visual mesh filename=robotiq_2f_85_gripper_visualization/meshes/visual/base_link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
Joints:
- added joint gripper_joint: type revolute, parent wrist_3_link, child gripper_link, origin xyz=0 0 0 rpy=0 0 90, limit lower=0 upper=0.8 effort=1000 velocity=0.5

Commit message: testing on this branch

File: content/assets/urdf/robot_info/robot.urdf (robot description, URDF)
Before this commit: robot ur, 22 links, 21 joints
Links:
- removed link robotiq_arg2f_base_link
- added link gripper_link, mass 0.7; collision mesh filename=robotiq_2f_85_gripper_visualization/meshes/collision/base_l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; visual mesh filename=robotiq_2f_85_gripper_visualization/meshes/visual/base_link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
Joints:
- joint gripper_main_joint: child robotiq_arg2f_base_link -> gripper_link
- joint left_outer_knuckle_joint: parent robotiq_arg2f_base_link -> gripper_link
- joint left_proximal_phalanx_joint: parent robotiq_arg2f_base_link -> gripper_link
- joint right_outer_knuckle_joint: parent robotiq_arg2f_base_link -> gripper_link
- joint right_proximal_phalanx_joint: parent robotiq_arg2f_base_link -> gripper_link

File: content/assets/urdf/robot_info/robot_storm.urdf (robot description, URDF)
Before this commit: robot ur, 8 links, 7 joints
Joints:
- joint gripper_joint: type revolute -> fixed

Commit message: Keep running test

File: content/assets/urdf/robot_info/robot.urdf (robot description, URDF)
Before this commit: robot ur, 13 links, 12 joints
Links:
- added link left_bar, mass 0.022614240507152; collision mesh filename=robotiq_2f_85_gripper_visualization/meshes/collision/bar.stl; visual mesh filename=robotiq_2f_85_gripper_visualization/meshes/visual/bar.stl
- added link left_distal_phalanx, mass 0.0104003125914103; collision mesh filename=robotiq_2f_85_gripper_visualization/meshes/collision/distal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; visual mesh filename=robotiq_2f_85_gripper_visualization/meshes/visual/distal_ph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
- added link left_outer_knuckle, mass 0.00853198276973456; collision mesh filename=robotiq_2f_85_gripper_visualization/meshes/collision/outer_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; visual mesh filename=robotiq_2f_85_gripper_visualization/meshes/visual/outer_knu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
- added link left_proximal_phalanx, mass 0.0271177346495152; collision mesh filename=robotiq_2f_85_gripper_visualization/meshes/collision/proxim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; visual mesh filename=robotiq_2f_85_gripper_visualization/meshes/visual/proximal_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
- added link right_bar, mass 0.022614240507152; collision mesh filename=robotiq_2f_85_gripper_visualization/meshes/collision/bar.stl; visual mesh filename=robotiq_2f_85_gripper_visualization/meshes/visual/bar.stl
- added link right_distal_phalanx, mass 0.0104003125914103; collision mesh filename=robotiq_2f_85_gripper_visualization/meshes/collision/distal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; visual mesh filename=robotiq_2f_85_gripper_visualization/meshes/visual/distal_ph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
- added link right_outer_knuckle, mass 0.00853198276973456; collision mesh filename=robotiq_2f_85_gripper_visualization/meshes/collision/outer_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; visual mesh filename=robotiq_2f_85_gripper_visualization/meshes/visual/outer_knu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
- added link right_proximal_phalanx, mass 0.0271177346495152; collision mesh filename=robotiq_2f_85_gripper_visualization/meshes/collision/proxim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; visual mesh filename=robotiq_2f_85_gripper_visualization/meshes/visual/proximal_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
- added link robotiq_arg2f_base_link, mass 0.7; collision mesh filename=robotiq_2f_85_gripper_visualization/meshes/collision/base_l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; visual mesh filename=robotiq_2f_85_gripper_visualization/meshes/visual/base_link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
Joints:
- added joint gripper_main_joint: type fixed, parent wrist_3_link, child robotiq_arg2f_base_link, origin xyz=0 0 0 rpy=0 0 90
- added joint left_bar_joint: type fixed, parent left_distal_phalanx, child left_bar, origin xyz=0 0.0315 -0.0041 rpy=0 0 0, axis 1 0 0
- added joint left_distal_phalanx_joint: type fixed, parent left_proximal_phalanx, child left_distal_phalanx, origin xyz=0 0.0061 0.0471 rpy=0 0 0, axis 0 0 0, limit lower=-0.8757 upper=0 effort=1000 velocity=0.5, mimic joint=left_outer_knuckle_joint multiplier=-1 offset=0
- added joint left_outer_knuckle_joint: type fixed, parent robotiq_arg2f_base_link, child left_outer_knuckle, origin xyz=0 -0.0306011 0.054904 rpy=0 0 3.141592653589793, axis 0 0 0, limit lower=0 upper=0.8 effort=1000 velocity=0.5
- added joint left_proximal_phalanx_joint: type fixed, parent robotiq_arg2f_base_link, child left_proximal_phalanx, origin xyz=0 -0.0127 0.06142 rpy=.125 0 3.141592653589793, axis 1 0 0, limit lower=0 upper=0.8757 effort=1000 velocity=0.5, mimic joint=left_outer_knuckle_joint multiplier=1 offset=0
- added joint right_bar_joint: type fixed, parent right_distal_phalanx, child right_bar, origin xyz=0 0.0315 -0.0041 rpy=0 0 0, axis 1 0 0
- added joint right_distal_phalanx_joint: type fixed, parent right_proximal_phalanx, child right_distal_phalanx, origin xyz=0 0.0061 0.0471 rpy=0 0 0, axis 1 0 0, limit lower=-0.8757 upper=0 effort=1000 velocity=0.5, mimic joint=left_outer_knuckle_joint multiplier=-1 offset=0
- added joint right_outer_knuckle_joint: type fixed, parent robotiq_arg2f_base_link, child right_outer_knuckle, origin xyz=0 0.0306011 0.054904 rpy=0 0 0, axis 1 0 0, limit lower=0 upper=0.81 effort=1000 velocity=0.5, mimic joint=left_outer_knuckle_joint multiplier=1 offset=0
- added joint right_proximal_phalanx_joint: type fixed, parent robotiq_arg2f_base_link, child right_proximal_phalanx, origin xyz=0 0.0127 0.06142 rpy=.125 0 0.0, axis 1 0 0, limit lower=0 upper=0.8757 effort=1000 velocity=0.5, mimic joint=left_outer_knuckle_joint multiplier=1 offset=0

File: content/assets/urdf/robot_info/robot_storm.urdf (robot description, URDF)
Before this commit: robot ur, 7 links, 6 joints
Links:
- added link gripper_link, mass 0.7; collision mesh filename=robotiq_2f_85_gripper_visualization/meshes/collision/base_l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; visual mesh filename=robotiq_2f_85_gripper_visualization/meshes/visual/base_link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
Joints:
- added joint gripper_joint: type fixed, parent wrist_3_link, child gripper_link, origin xyz=0 0 0 rpy=0 0 90, limit lower=0 upper=0.8 effort=1000 velocity=0.5
